File: TreadmillDaughterboard.kicad_sch (KiCad schematic)
At the start: 21 parts, among them J10 Conn_01x03_Socket, J7 RJ45, SW2 SW_Push_Open_Dual, SW3 SW_Push_Open_Dual

Commit message: Fixed Daughterboard Outputs Box
Replaced the TM hierarchical boxes with connectors
Parts:
- renumbered C13 to C17, C14 to C18, D7 to D13, D5 to D14, D6 to D15, J7 to J13, J10 to J14, R13 to R21, R10 to R22, R11 to R23, R12 to R24, SW3 to SW7, SW2 to SW8, TP14 to TP30, TP7 to TP31, TP8 to TP32, TP9 to TP33, TP10 to TP34, TP11 to TP35, TP12 to TP36, TP13 to TP37

Commit message: Relay work
did all the relay related work
Parts:
- added C13: .1UF, symbol Device:C
- added J15: Conn_01x03_Socket, symbol Connector:Conn_01x03_Socket
- added U3: DRV5033AJQLPGM, Package_TO_SOT_THT:TO-92_Inline, symbol Sensor_Magnetic:DRV5033AJxLPG
- R24: now fitted
Connections:
- net GND: now also C13.2
- new net: C13.1, J15.1 (Pin_1), U3.1 (VCC)
- new net: J15.2 (Pin_2), U3.2 (GND)
- new net: J15.3 (Pin_3), U3.3 (OUT)
Other:
- note added: "HALL DAUGHTERBOARD"
- title: (none) -> TIME MACHINE DAUGHTERBOARD
- moved on the sheet: J14, TP30, TP31, TP32, TP33, TP34, TP35, TP36, TP37
