File: Kicad/FluxCapacitor.kicad_sch (KiCad schematic)
At the start: 118 parts, among them J1 Barrel_Jack, J10 RELAY, J19 Conn_01x03_Socket, J2 TM_1, J20 Conn_01x03_Socket, J21 Conn_01x03_Socket, J22 Conn_01x03_Socket, J23 Conn_01x03_Socket, J3 TM_2, J4 Conn_01x02, J7 TM_1, J8 TM_1, J9 RELAY, K1 G5V-1, M1 SYS_FAN, Q1 2N7000, Q2 IRF4905PBF, Q3 2N7000, Q4 2N7000, SW1 SW_SPDT_321, SW9 SW_Push_Open_Dual, U1 OKI-78SR-5_1.5-W36-C, U2 ESP32_DEVBOARD, U6 SMF5.0A-T13

Commit message: Added footprints, started assigning
-Changed Buzzer and Led matrix to run off of 5v_Raw to avoid getting backfed when usb is plugged into esp32
-added all footprints to library
-started assigning footprints
Parts:
- C1, C3, C9: footprint (none) -> FluxCapacitor:25YXJ100M5X11
- C10, C12, C19, C2, C21, C24, C4, C5, C6, C7: footprint (none) -> FluxCapacitor:CC0805KRX7R9BB104
- C11, C20: footprint (none) -> FluxCapacitor:GMC21X7R106K25NT
- C8: footprint (none) -> FluxCapacitor:PHV-5R4V155-R
- D1: footprint 1N4744A:DIOAD1036W78L463D237 -> FluxCapacitor:1N4744A
- renumbered U_BTN_EXPANDER to U_BTN_EXPANDER1
Connections:
- net 5V_RAW: now also BZ1.1 (+), C19.2
- net 5V_SYS: no longer BZ1.1 (+), C19.2
Changed lines of the file:
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@@
 			)
 		)
-		(property "Footprint" ""
+		(property "Footprint" "FluxCapacitor:CC0805KRX7R9BB104"
 			(at 236.5248 146.05 0)
 			(hide yes)
@@
 	(symbol
 		(lib_id "power:+12V")
+		(at 238.76 59.69 270)
+		(unit 1)
+		(body_style 1)
+		(exclude_from_sim no)
+		(in_bom yes)
+		(on_board yes)
+		(in_pos_files yes)
+		(dnp no)
+		(property "Reference" "#PWR086"
+			(at 234.95 59.69 0)
+			(hide yes)
+			(show_name no)
+			(do_not_autoplace no)
+			(effects
+				(font
+					(size 1.27 1.27)
+				)
+			)
+		)
+		(property "Value" "5V_RAW"
+			(at 248.92 59.69 90)
+			(show_name no)
+			(do_not_autoplace no)
+			(effects
+				(font
+					(size 1.27 1.27)
+				)
+				(justify right)
+			)
+		)
+		(property "Footprint" ""
+			(at 238.76 59.69 0)
+			(hide yes)
+			(show_name no)
+			(do_not_autoplace no)
+			(effects
+				(font
+					(size 1.27 1.27)
+				)
+			)
+		)
+		(property "Datasheet" ""
+			(at 238.76 59.69 0)
+			(hide yes)
+			(show_name no)
+			(do_not_autoplace no)
+			(effects
+				(font
+					(size 1.27 1.27)
+				)
+			)
+		)
+		(property "Description" "Power symbol creates a global label with name \"+12V\""
+			(at 238.76 59.69 0)
+			(hide yes)
+			(show_name no)
+			(do_not_autoplace no)
+			(effects
+				(font
+					(size 1.27 1.27)
+				)
+			)
+		)
+		(pin "1"
+		)
+		(instances
+			(project "FluxCapacitor"
+				(path "/feb6d8df-599a-4f82-8f89-f7a3c96de191"
+					(reference "#PWR086")
+					(unit 1)
+				)
+			)
+		)
+	)
+	(symbol
+		(lib_id "power:+12V")
 		(at 200.66 118.11 90)
 		(unit 1)
@@
 			)
 		)
-		(property "Footprint" ""
+		(property "Footprint" "FluxCapacitor:25YXJ100M5X11"
 			(at 138.1252 96.52 0)
 			(hide yes)
@@
 			)
 		)
-		(property "Footprint" ""
+		(property "Footprint" "FluxCapacitor:CC0805KRX7R9BB104"
 			(at 40.3352 134.62 0)
 			(hide yes)
@@
 			)
 		)
-		(property "Footprint" ""
+		(property "Footprint" "FluxCapacitor:CC0805KRX7R9BB104"
 			(at 57.15 52.3748 0)
 			(hide yes)
@@
 			)
 		)
-		(property "Footprint" ""
+		(property "Footprint" "FluxCapacitor:25YXJ100M5X11"
 			(at 97.79 52.3748 0)
 			(hide yes)
@@
 			)
 		)
-		(property "Value" "5V_SYS"
+		(property "Value" "5V_RAW"
 			(at 86.36 71.628 90)
 			(show_name no)
@@
 			)
 		)
-		(property "Footprint" ""
+		(property "Footprint" "FluxCapacitor:CC0805KRX7R9BB104"
 			(at 251.7648 80.01 0)
 			(hide yes)
@@
 			)
 		)
-		(property "Footprint" ""
+		(property "Footprint" "FluxCapacitor:CC0805KRX7R9BB104"
 			(at 147.0152 96.52 0)
 			(hide yes)
@@
 			)
 		)
-		(property "Footprint" ""
+		(property "Footprint" "FluxCapacitor:GMC21X7R106K25NT"
 			(at 89.8652 116.84 0)
 			(hide yes)
@@
 			)
 		)
-		(property "Footprint" ""
+		(property "Footprint" "FluxCapacitor:CC0805KRX7R9BB104"
 			(at 39.0652 76.2 0)
 			(hide yes)
@@
 			)
 		)
-		(property "Footprint" ""
+		(property "Footprint" "FluxCapacitor:CC0805KRX7R9BB104"
 			(at 97.4852 116.84 0)
 			(hide yes)
@@
 			)
 		)
-		(property "Footprint" ""
+		(property "Footprint" "FluxCapacitor:25YXJ100M5X11"
 			(at 57.15 39.6748 0)
 			(hide yes)
@@
 			)
 		)
-		(property "Footprint" ""
+		(property "Footprint" "FluxCapacitor:PHV-5R4V155-R"
 			(at 118.11 98.7552 0)
 			(hide yes)
@@
 			)
 		)
-		(property "Footprint" ""
+		(property "Footprint" "FluxCapacitor:GMC21X7R106K25NT"
 			(at 240.3348 80.01 0)
 			(hide yes)
@@
 			)
 		)
-		(property "Footprint" ""
+		(property "Footprint" "FluxCapacitor:CC0805KRX7R9BB104"
 			(at 92.4052 77.47 0)
 			(hide yes)
@@
 		(dnp no)
 		(fields_autoplaced yes)
-		(property "Reference" "U_BTN_EXPANDER"
+		(property "Reference" "U_BTN_EXPANDER1"
 			(at 45.3233 134.62 0)
 			(show_name no)
@@
 			(project "FluxCapacitor"
 				(path "/feb6d8df-599a-4f82-8f89-f7a3c96de191"
-					(reference "U_BTN_EXPANDER")
+					(reference "U_BTN_EXPANDER1")
 					(unit 1)
 				)
@@
 			)
 		)
-		(property "Footprint" ""
+		(property "Footprint" "FluxCapacitor:CC0805KRX7R9BB104"
 			(at 77.47 48.5648 0)
 			(hide yes)
@@
 			)
 		)
-		(property "Footprint" ""
+		(property "Footprint" "FluxCapacitor:CC0805KRX7R9BB104"
 			(at 97.79 40.9448 0)
 			(hide yes)
@@
 	)
 	(symbol
-		(lib_id "power:+12V")
-		(at 238.76 59.69 270)
-		(unit 1)
-		(body_style 1)
-		(exclude_from_sim no)
-		(in_bom yes)
-		(on_board yes)
-		(in_pos_files yes)
-		(dnp no)
-		(fields_autoplaced yes)
-		(property "Reference" "#PWR086"
-			(at 234.95 59.69 0)
-			(hide yes)
-			(show_name no)
-			(do_not_autoplace no)
-			(effects
-				(font
-					(size 1.27 1.27)
-				)
-			)
-		)
-		(property "Value" "5V_SYS"
-			(at 242.57 59.6899 90)
-			(show_name no)
-			(do_not_autoplace no)
-			(effects
-				(font
-					(size 1.27 1.27)
-				)
-				(justify left)
-			)
-		)
-		(property "Footprint" ""
-			(at 238.76 59.69 0)
-			(hide yes)
-			(show_name no)
-			(do_not_autoplace no)
-			(effects
-				(font
-					(size 1.27 1.27)
-				)
-			)
-		)
-		(property "Datasheet" ""
-			(at 238.76 59.69 0)
-			(hide yes)
-			(show_name no)
-			(do_not_autoplace no)
-			(effects
-				(font
-					(size 1.27 1.27)
-				)
-			)
-		)
-		(property "Description" "Power symbol creates a global label with name \"+12V\""
-			(at 238.76 59.69 0)
-			(hide yes)
-			(show_name no)
-			(do_not_autoplace no)
-			(effects
-				(font
-					(size 1.27 1.27)
-				)
-			)
-		)
-		(pin "1"
-		)
-		(instances
-			(project "FluxCapacitor"
-				(path "/feb6d8df-599a-4f82-8f89-f7a3c96de191"
-					(reference "#PWR086")
-					(unit 1)
-				)
-			)
-		)
-	)
-	(symbol
 		(lib_id "Switch:SW_Push_Open_Dual")
 		(at 242.57 128.27 0)
@@
 			)
 		)
-		(property "Footprint" "1N4744A:DIOAD1036W78L463D237"
+		(property "Footprint" "FluxCapacitor:1N4744A"
 			(at 30.48 50.8 0)
 			(hide yes)
