File: Kicad/FluxCapacitor.kicad_sch (KiCad schematic)
At the start: 118 parts, among them J1 Barrel_Jack, J10 RELAY, J19 Conn_01x03_Socket, J2 TM_1, J20 Conn_01x03_Socket, J21 Conn_01x03_Socket, J22 Conn_01x03_Socket, J23 Conn_01x03_Socket, J3 TM_2, J4 Conn_01x02, J7 TM_1, J8 TM_1, J9 RELAY, K1 G5V-1, M1 SYS_FAN, Q1 2N7000, Q2 IRF4905PBF, Q3 2N7000, Q4 2N7000, SW1 SW_SPDT_321, SW9 SW_Push_Open_Dual, U1 OKI-78SR-5_1.5-W36-C, U2 ESP32_DEVBOARD, U6 SMF5.0A-T13

Commit message: All footprints assigned
All footprints assigned
Parts:
- BZ1: footprint (none) -> FluxCapacitor:PT2040PQ
- D10, D11, D12, D16, D17, D18, D19, D6, D8, D9: footprint (none) -> FluxCapacitor:LED_0805_2012Metric_Pad1.15x1.40mm_HandSolder
- D4: footprint Diode_SMD:Nexperia_DSN1608-2_1.6x0.8mm -> FluxCapacitor:P6KE15A
- D5: footprint Diode_THT:D_DO-35_SOD27_P7.62mm_Horizontal -> FluxCapacitor:1N4148
- F1: value 1 A Polyfuse -> MF-R110; footprint (none) -> FluxCapacitor:MF-R110
- J1: value Barrel_Jack -> PJ-002A; footprint (none) -> FluxCapacitor:PJ-002A
- J10, J9: footprint (none) -> FluxCapacitor:SS-6488-NF-50
- J19, J20, J21, J22, J23: value Conn_01x03_Socket -> JST_PH_01x03_Socket; footprint (none) -> FluxCapacitor:JST_PH_B3B-PH-K_1x03_P2.00mm_Vertical
- J2, J3: footprint (none) -> FluxCapacitor:JST_PH_B3B-PH-K_1x03_P2.00mm_Vertical
- J4: value Conn_01x02 -> TREADMILL_CTRL_PANEL1; footprint (none) -> FluxCapacitor:PinHeader_1x02_P2.54mm_Vertical
- J7: value TM_1 -> TM_4; footprint (none) -> FluxCapacitor:JST_PH_B3B-PH-K_1x03_P2.00mm_Vertical
- J8: value TM_1 -> TM_2; footprint (none) -> FluxCapacitor:JST_PH_B3B-PH-K_1x03_P2.00mm_Vertical
- JP1, JP2, JP3: footprint (none) -> FluxCapacitor:SolderJumper-2_P1.3mm_Open_Pad1.0x1.5mm
- M1: footprint (none) -> FluxCapacitor:FanPinHeader_1x04_P2.54mm_Vertical
- Q1, Q3, Q4: footprint Q_TO-92_135AN_OSI -> FluxCapacitor:2N7000
- Q2: footprint TO254P469X1042X1967-3P -> FluxCapacitor:IRF4905PBF
- R1, R10, R11, R12, R16, R17, R18, R19, R2, R20, R25, R26, R27, R28, R29, R3, R30, R31, R32, R33, R34, R35, R36, R37, R4, R5, R6, R7, R8, R9: footprint (none) -> FluxCapacitor:R_0805_2012Metric_Pad1.20x1.40mm_HandSolder
- SW1: footprint (none) -> FluxCapacitor:TM SPDT switch
- SW9: footprint (none) -> FluxCapacitor:D6R60F1LFS
- TP1, TP10, TP11, TP12, TP13, TP14, TP15, TP16, TP17, TP18, TP19, TP2, TP20, TP21, TP22, TP23, TP24, TP25, TP3, TP4, TP5, TP6, TP8, TP9: footprint (none) -> FluxCapacitor:TestPoint_Pad_D2.0mm
- TP7: value TP_TX -> TP_RX; footprint (none) -> FluxCapacitor:TestPoint_Pad_D2.0mm
- U2: footprint (none) -> FluxCapacitor:ESP32 DEVBOARD
- U6: footprint (none) -> FluxCapacitor:SMF5.0A-T13
Connections:
- net at C3.1, C4.1, TP2.1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: now also JP2.1 (A)
