File: Kicad/FAULT_LEDS.kicad_sch (KiCad schematic)
At the start: 9 parts, among them U4 HT16K33_DEVBOARD, U5 PCA9306DCUR

Commit message: Finished schematic
Other:
- title: (none) -> FAULT LEDS
Changed lines of the file:
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@@
 	(generator_version "10.0")
 	(paper "A4")
+	(title_block
+		(title "FAULT LEDS")
+	)
 	(junction
 		(at 100.33 105.41)

Commit message: Touchups
Parts:
- C14: value .1UF -> 0.1UF
- C15: symbol Device:C_Polarized -> Device:C
- R13, R14: value 4.7k -> 4.7K
Changed lines of the file:
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@@
 			)
 		)
-		(property "Value" "4.7k"
+		(property "Value" "4.7K"
 			(at 113.538 96.774 90)
 			(show_name no)
@@
 			)
 		)
-		(property "Value" "4.7k"
+		(property "Value" "4.7K"
 			(at 102.616 110.998 90)
 			(show_name no)
@@
 			)
 		)
-		(property "Value" ".1UF"
+		(property "Value" "0.1UF"
 			(at 114.3 111.252 90)
 			(show_name no)
@@
 	)
 	(symbol
-		(lib_id "Device:C_Polarized")
+		(lib_id "Device:C")
 		(at 114.3 115.57 90)
 		(unit 1)
@@
 		(dnp no)
 		(property "Reference" "C15"
-			(at 117.348 114.046 90)
-			(show_name no)
-			(do_not_autoplace no)
-			(effects
-				(font
-					(size 1.27 1.27)
-				)
-			)
-		)
+			(at 116.332 120.904 90)
+			(show_name no)
+			(do_not_autoplace no)
+			(effects
+				(font
+					(size 1.27 1.27)
+				)
+				(justify left)
+			)
+		)

Commit message: Added footprints, started assigning
-Changed Buzzer and Led matrix to run off of 5v_Raw to avoid getting backfed when usb is plugged into esp32
-added all footprints to library
-started assigning footprints
Parts:
- C14: footprint (none) -> FluxCapacitor:CC0805KRX7R9BB104
- C15: footprint (none) -> FluxCapacitor:GMC21X7R106K25NT
- C16: footprint (none) -> FluxCapacitor:C0805C101J5GACTU
Changed lines of the file:
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@@
 	(hierarchical_label "GND"
 		(shape input)
-		(at 128.27 73.66 180)
+		(at 139.7 88.9 180)
 		(effects
 			(font
@@
 	(symbol
 		(lib_id "power:GND")
-		(at 128.27 73.66 90)
+		(at 139.7 88.9 90)
 		(unit 1)
 		(body_style 1)
@@
 		(fields_autoplaced yes)
 		(property "Reference" "#PWR032"
-			(at 134.62 73.66 0)
+			(at 146.05 88.9 0)
 			(hide yes)
 			(show_name no)
@@
 		)
 		(property "Value" "GND"
-			(at 132.08 73.6599 90)
+			(at 143.51 88.8999 90)
 			(show_name no)
 			(do_not_autoplace no)
@@
 		)
 		(property "Footprint" ""
-			(at 128.27 73.66 0)
+			(at 139.7 88.9 0)
 			(hide yes)
 			(show_name no)
@@
 		)
 		(property "Datasheet" ""
-			(at 128.27 73.66 0)
+			(at 139.7 88.9 0)
 			(hide yes)
 			(show_name no)
@@
 		)
 		(property "Description" "Power symbol creates a global label with name \"GND\" , ground"
-			(at 128.27 73.66 0)
+			(at 139.7 88.9 0)
 			(hide yes)
 			(show_name no)
@@
 			)
 		)
-		(property "Footprint" ""
+		(property "Footprint" "FluxCapacitor:CC0805KRX7R9BB104"
 			(at 118.11 106.9848 0)
 			(hide yes)
@@
 			)
 		)
-		(property "Footprint" ""
+		(property "Footprint" "FluxCapacitor:C0805C101J5GACTU"
 			(at 101.2952 92.71 0)
 			(hide yes)
@@
 			)
 		)
-		(property "Footprint" ""
+		(property "Footprint" "FluxCapacitor:GMC21X7R106K25NT"
 			(at 118.11 114.6048 0)
 			(hide yes)

Commit message: All footprints assigned
All footprints assigned
Parts:
- LED1: footprint RLA18_DC56-11EWA_KNB -> FluxCapacitor:DC56-11EWA
- R13, R14, R15: footprint (none) -> FluxCapacitor:R_0805_2012Metric_Pad1.20x1.40mm_HandSolder
- U4: footprint (none) -> FluxCapacitor:HT16K33 DEVBOARD
- U5: footprint PCA9306DCUR:SOP50P310X90-8N -> FluxCapacitor:PCA9306DCUR
Changed lines of the file:
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@@
 			)
 		)
-		(property "Footprint" ""
+		(property "Footprint" "FluxCapacitor:R_0805_2012Metric_Pad1.20x1.40mm_HandSolder"
 			(at 115.57 97.282 90)
 			(hide yes)
@@
 			)
 		)
-		(property "Footprint" ""
+		(property "Footprint" "FluxCapacitor:R_0805_2012Metric_Pad1.20x1.40mm_HandSolder"
 			(at 98.552 109.22 90)
 			(hide yes)
@@
 			)
 		)
-		(property "Footprint" "PCA9306DCUR:SOP50P310X90-8N"
+		(property "Footprint" "FluxCapacitor:PCA9306DCUR"
 			(at 80.01 100.33 0)
 			(hide yes)
@@
 			)
 		)
-		(property "Footprint" ""
+		(property "Footprint" "FluxCapacitor:HT16K33 DEVBOARD"
 			(at 140.97 115.57 0)
 			(hide yes)
@@
 			)
 		)
-		(property "Footprint" "RLA18_DC56-11EWA_KNB"
+		(property "Footprint" "FluxCapacitor:DC56-11EWA"
 			(at 186.69 87.63 0)
 			(hide yes)
@@
 			)
 		)
-		(property "Footprint" ""
+		(property "Footprint" "FluxCapacitor:R_0805_2012Metric_Pad1.20x1.40mm_HandSolder"
 			(at 115.57 94.488 90)
 			(hide yes)
