File: Kicad/TreadmillDaughterboard.kicad_sch (KiCad schematic)
At the start: 24 parts, among them J13 RJ45, J14 Conn_01x03_Socket, J15 Conn_01x03_Socket, SW7 SW_Push_Open_Dual, SW8 SW_Push_Open_Dual, U3 DRV5033AJQLPGM

Commit message: Finished Schematic
   did
-All debugging leds
-buzzer
-ran ERC

to do
-fix ERC problems

it is
-too late lol
Parts:
- C18: value C_Polarized -> 10UF
Changed lines of the file:
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@@
 		(dnp no)
 		(property "Reference" "C18"
-			(at 42.545 43.18 0)
+			(at 44.45 46.228 0)
 			(show_name no)
 			(do_not_autoplace no)
@@
 			)
 		)
-		(property "Value" "C_Polarized"
+		(property "Value" "10UF"
 			(at 42.545 48.26 0)
 			(show_name no)

Commit message: Finished schematic
Parts:
- added C22, C23: .1UF, symbol Device:C
- R21, R22, R23: value 1.5k -> 680Ω
- U3: value DRV5033AJQLPGM -> DRV5033AJxLPG
Connections:
- net GND: now also C22.1, C23.1
- net PRESET_BTN: now also C22.2
- net STARTSTOP_BTN: now also C23.2
- net TDB_3V3 renamed TBD_3V3
Other:
- moved on the sheet: C13, C17, C18, J14, J15, R24, SW7, SW8, U3

Commit message: Touchups
Parts:
- C13, C22, C23: value .1UF -> 0.1UF
- C17: value .1uf -> 0.1UF
- C18: symbol Device:C_Polarized -> Device:C
Changed lines of the file:
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@@
 			)
 		)
-		(property "Value" ".1uf"
-			(at 30.734 49.53 0)
+		(property "Value" "0.1UF"
+			(at 29.464 49.784 0)
 			(show_name no)
 			(do_not_autoplace no)
@@
 	)
 	(symbol
-		(lib_id "Device:C_Polarized")
+		(lib_id "Device:C")
 		(at 40.64 45.72 0)
 		(unit 1)
@@
 		(dnp no)
 		(property "Reference" "C18"
-			(at 43.18 46.228 0)
+			(at 43.18 46.482 0)
 			(show_name no)
 			(do_not_autoplace no)
@@
 			)
 		)
-		(property "Description" "Polarized capacitor"
+		(property "Description" "Unpolarized capacitor"
 			(at 40.64 45.72 0)
 			(hide yes)
@@
 			)
 		)
-		(property "Value" ".1UF"
+		(property "Value" "0.1UF"
 			(at 36.576 86.36 0)
 			(show_name no)
@@
 			)
 		)
-		(property "Value" ".1UF"
+		(property "Value" "0.1UF"
 			(at 78.74 50.038 0)
 			(show_name no)
@@
 			)
 		)
-		(property "Value" ".1UF"
+		(property "Value" "0.1UF"
 			(at 36.576 96.52 0)
 			(show_name no)

Commit message: DNP the TM switch
Parts:
- SW8: now not fitted
Changed lines of the file:
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@@
 		(on_board yes)
 		(in_pos_files yes)
-		(dnp no)
+		(dnp yes)
 		(property "Reference" "SW8"
 			(at 46.99 97.79 0)

Commit message: Added footprints, started assigning
-Changed Buzzer and Led matrix to run off of 5v_Raw to avoid getting backfed when usb is plugged into esp32
-added all footprints to library
-started assigning footprints
Parts:
- C13, C17, C22, C23: footprint (none) -> FluxCapacitor:CC0805KRX7R9BB104
- C18: footprint (none) -> FluxCapacitor:GMC21X7R106K25NT
Changed lines of the file:
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@@
 			)
 		)
-		(property "Footprint" ""
+		(property "Footprint" "FluxCapacitor:CC0805KRX7R9BB104"
 			(at 36.5252 49.53 0)
 			(hide yes)
@@
 			)
 		)
-		(property "Footprint" ""
+		(property "Footprint" "FluxCapacitor:GMC21X7R106K25NT"
 			(at 41.6052 49.53 0)
 			(hide yes)
@@
 			)
 		)
-		(property "Footprint" ""
+		(property "Footprint" "FluxCapacitor:CC0805KRX7R9BB104"
 			(at 38.4048 83.82 0)
 			(hide yes)
@@
 			)
 		)
-		(property "Footprint" ""
+		(property "Footprint" "FluxCapacitor:CC0805KRX7R9BB104"
 			(at 77.1652 50.8 0)
 			(hide yes)
@@
 			)
 		)
-		(property "Footprint" ""
+		(property "Footprint" "FluxCapacitor:CC0805KRX7R9BB104"
 			(at 38.4048 93.98 0)
 			(hide yes)

Commit message: All footprints assigned
All footprints assigned
Parts:
- C23: now not fitted
- D13: value RED LED -> RED TM LED; footprint (none) -> FluxCapacitor:LED_D5.0mm
- D14, D15: value GREEN LED -> GREEN TM LED; footprint (none) -> FluxCapacitor:LED_D5.0mm
- J13: footprint (none) -> FluxCapacitor:SS-6488-NF-50
- J14, J15: footprint (none) -> FluxCapacitor:JST_PH_B3B-PH-K_1x03_P2.00mm_Vertical
- R21, R22, R23, R24: footprint (none) -> FluxCapacitor:R_0805_2012Metric_Pad1.20x1.40mm_HandSolder
- SW7, SW8: footprint (none) -> FluxCapacitor:D6R60F1LFS
- TP30, TP31, TP32, TP33, TP34, TP35, TP36, TP37: footprint (none) -> FluxCapacitor:TestPoint_Pad_D2.0mm
Changed lines of the file:
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@@
 	)
 	(junction
-		(at 48.26 71.12)
-		(diameter 0)
-		(color 0 0 0 0)
-	)
-	(junction
 		(at 39.37 100.33)
 		(diameter 0)
@@
 	(wire
 		(pts
-			(xy 48.26 71.12) (xy 52.07 71.12)
+			(xy 48.26 67.31) (xy 52.07 67.31)
 		)
 		(stroke
@@
 	(wire
 		(pts
-			(xy 48.26 71.12) (xy 48.26 73.66)
-		)
-		(stroke
-			(width 0)
-			(type default)
-		)
-	)
-	(wire
-		(pts
 			(xy 68.58 43.18) (xy 76.2 43.18)
 		)
@@
 	(wire
 		(pts
-			(xy 48.26 67.31) (xy 48.26 71.12)
+			(xy 48.26 67.31) (xy 48.26 73.66)
 		)
 		(stroke
@@
 		)
 	)
+	(wire
+		(pts
+			(xy 52.07 67.31) (xy 52.07 71.12)
+		)
+		(stroke
+			(width 0)
+			(type default)
+		)
+	)
 	(label "PRESET_BTN"
 		(at 31.75 85.09 180)
@@
 			)
 		)
-		(property "Footprint" ""
+		(property "Footprint" "FluxCapacitor:TestPoint_Pad_D2.0mm"
 			(at 31.75 137.16 0)
 			(hide yes)
@@
 			)
 		)
-		(property "Footprint" ""
+		(property "Footprint" "FluxCapacitor:TestPoint_Pad_D2.0mm"
 			(at 31.75 114.3 0)
 			(hide yes)
@@
 			)
 		)
-		(property "Footprint" ""
+		(property "Footprint" "FluxCapacitor:R_0805_2012Metric_Pad1.20x1.40mm_HandSolder"
 			(at 34.29 75.438 90)
 			(hide yes)
@@
 			)
 		)
-		(property "Footprint" ""
+		(property "Footprint" "FluxCapacitor:TestPoint_Pad_D2.0mm"
 			(at 31.75 127 0)
 			(hide yes)
@@
 			)
 		)
-		(property "Footprint" ""
+		(property "Footprint" "FluxCapacitor:JST_PH_B3B-PH-K_1x03_P2.00mm_Vertical"
 			(at 63.5 40.64 0)
 			(hide yes)
@@
 			)
 		)
-		(property "Footprint" ""
+		(property "Footprint" "FluxCapacitor:SS-6488-NF-50"
 			(at 25.4 33.655 90)
 			(hide yes)
@@
 			)
 		)
-		(property "Footprint" ""
+		(property "Footprint" "FluxCapacitor:TestPoint_Pad_D2.0mm"
 			(at 31.75 142.24 0)
 			(hide yes)
@@
 			)
 		)
-		(property "Footprint" ""
+		(property "Footprint" "FluxCapacitor:TestPoint_Pad_D2.0mm"
 			(at 31.75 132.08 0)
 			(hide yes)
@@
 			)
 		)
-		(property "Footprint" ""
+		(property "Footprint" "FluxCapacitor:TestPoint_Pad_D2.0mm"
 			(at 31.75 116.84 0)
 			(hide yes)
@@
 			)
 		)
-		(property "Footprint" ""
+		(property "Footprint" "FluxCapacitor:TestPoint_Pad_D2.0mm"
 			(at 31.75 119.38 0)
 			(hide yes)
@@
 			)
 		)
-		(property "Value" "GREEN LED"
+		(property "Value" "GREEN TM LED"
 			(at 40.386 69.85 0)
 			(show_name no)
@@
 			)
 		)
-		(property "Footprint" ""
+		(property "Footprint" "FluxCapacitor:LED_D5.0mm"
 			(at 41.91 67.31 0)
 			(hide yes)
@@
 			)
 		)
-		(property "Value" "GREEN LED"
+		(property "Value" "GREEN TM LED"
 			(at 40.386 76.2 0)
 			(show_name no)
@@
 			)
 		)
-		(property "Footprint" ""
+		(property "Footprint" "FluxCapacitor:LED_D5.0mm"
 			(at 41.91 73.66 0)
 			(hide yes)
@@
 			)
 		)
-		(property "Footprint" ""
+		(property "Footprint" "FluxCapacitor:D6R60F1LFS"
 			(at 46.99 90.17 0)
 			(hide yes)
@@
 			)
 		)
-		(property "Footprint" ""
+		(property "Footprint" "FluxCapacitor:R_0805_2012Metric_Pad1.20x1.40mm_HandSolder"
 			(at 34.29 69.088 90)
 			(hide yes)
@@
 			)
 		)
-		(property "Footprint" ""
+		(property "Footprint" "FluxCapacitor:R_0805_2012Metric_Pad1.20x1.40mm_HandSolder"
 			(at 34.29 62.738 90)
 			(hide yes)
@@
 		(dnp no)
 		(property "Reference" "D13"
-			(at 39.116 61.976 0)
+			(at 38.862 61.976 0)
 			(show_name no)
 			(do_not_autoplace no)
@@
 			)
 		)
-		(property "Value" "RED LED"
+		(property "Value" "RED TM LED"
 			(at 40.386 63.5 0)
 			(show_name no)
@@
 			)
 		)
-		(property "Footprint" ""
+		(property "Footprint" "FluxCapacitor:LED_D5.0mm"
 			(at 41.91 60.96 0)
 			(hide yes)
@@
 			)
 		)
-		(property "Footprint" ""
+		(property "Footprint" "FluxCapacitor:JST_PH_B3B-PH-K_1x03_P2.00mm_Vertical"
 			(at 80.01 21.59 0)
 			(hide yes)
@@
 			)
 		)
-		(property "Footprint" ""
+		(property "Footprint" "FluxCapacitor:D6R60F1LFS"
 			(at 46.99 80.01 0)
 			(hide yes)
@@
 		(on_board yes)
 		(in_pos_files yes)
-		(dnp no)
+		(dnp yes)
 		(property "Reference" "C23"
 			(at 36.322 99.06 0)
@@
 			)
 		)
-		(property "Footprint" ""
+		(property "Footprint" "FluxCapacitor:TestPoint_Pad_D2.0mm"
 			(at 31.75 121.92 0)
 			(hide yes)
@@
 			)
 		)
-		(property "Footprint" ""
+		(property "Footprint" "FluxCapacitor:R_0805_2012Metric_Pad1.20x1.40mm_HandSolder"
 			(at 86.868 21.59 90)
 			(hide yes)
